Commit message: circle+square

File: scara_robot_left.urdf (robot description, URDF)
Before this commit: robot scara_robot_left, 9 links, 8 joints
Joints:
- joint rotation1: limit lower=-2.6 upper=2.6 effort=1000 velocity=1000 -> lower=-31.4 upper=31.4 effort=1000 velocity=1000
- joint rotation2: limit lower=-3.00 upper=3.00 effort=1000 velocity=1000 -> lower=-3 upper=3 effort=1000 velocity=1000
